Commit message: fix: use local meshes path for go2_x5
Co-authored-by: Copilot <copilot@github.com>

File: quadruped_manipulator/go2_x5/urdf/go2_x5.urdf (robot description, URDF)
Before this commit: robot go2, 38 links, 37 joints
Links:
- link FL_calf: geometry collision cylinder length=0.12 radius=0.012; visual mesh filename=../meshes/calf_0.obj
- link FL_foot: geometry collision sphere radius=0.022; visual mesh filename=../meshes/foot.obj
- link FL_hip: geometry collision cylinder length=0.04 radius=0.046; visual mesh filename=../meshes/hip_0.obj
- link FL_thigh: geometry collision box size=0.11 0.0245 0.034; visual mesh filename=../meshes/thigh_0.obj
- link FR_calf: geometry collision cylinder length=0.12 radius=0.013; visual mesh filename=../meshes/calf_mirror_0.obj
- link FR_foot: geometry collision sphere radius=0.022; visual mesh filename=../meshes/foot.obj
- link FR_hip: geometry collision cylinder length=0.04 radius=0.046; visual mesh filename=../meshes/hip_0.obj
- link FR_thigh: geometry collision box size=0.11 0.0245 0.034; visual mesh filename=../meshes/thigh_mirror_0.obj
- link RL_calf: geometry collision cylinder length=0.12 radius=0.013; visual mesh filename=../meshes/calf_0.obj
- link RL_foot: geometry collision sphere radius=0.022; visual mesh filename=../meshes/foot.obj
- link RL_hip: geometry collision cylinder length=0.04 radius=0.046; visual mesh filename=../meshes/hip_0.obj
- link RL_thigh: geometry collision box size=0.11 0.0245 0.034; visual mesh filename=../meshes/thigh_0.obj
- link RR_calf: geometry collision cylinder length=0.12 radius=0.013; visual mesh filename=../meshes/calf_mirror_0.obj
- link RR_foot: geometry collision sphere radius=0.022; visual mesh filename=../meshes/foot.obj
- link RR_hip: geometry collision cylinder length=0.04 radius=0.046; visual mesh filename=../meshes/hip_0.obj
- link RR_thigh: geometry collision box size=0.11 0.0245 0.034; visual mesh filename=../meshes/thigh_mirror_0.obj
- link base: geometry collision box size=0.3762 0.0935 0.114; visual mesh filename=../meshes/base_0.obj
- link link0: geometry collision cylinder length=0.06 radius=0.03; visual mesh filename=../meshes/base_link.obj
- link link1: geometry visual mesh filename=../meshes/link1.obj
- link link2: geometry collision box size=0.22 0.06 0.05; collision cylinder length=0.06 radius=0.03
- link link3: geometry collision box size=0.19 0.05 0.04; collision cylinder length=0.05 radius=0.028
- link link4: geometry collision cylinder length=0.04 radius=0.03; visual mesh filename=../meshes/link4.obj
- link link5: geometry collision cylinder length=0.04 radius=0.03; visual mesh filename=../meshes/link5.obj
- link link6: geometry collision cylinder length=0.06 radius=0.03; visual mesh filename=../meshes/link6.obj
- link link7: geometry collision box size=0.03 0.004 0.036; collision box size=0.04 0.004 0.0105
- link link8: geometry collision box size=0.03 0.004 0.036; collision box size=0.04 0.004 0.0105
