Commit message: feat: add go2_x5 model

File: quadruped_manipulator/go2_x5/urdf/go2_x5.urdf (robot description, URDF)
Before this commit: robot go2, 29 links, 28 joints
Links:
- added link link0, mass 0.43995; collision cylinder length=0.06 radius=0.03; visual mesh filename=../../../manipulator/x5/meshes/base_link.obj
- added link link1, mass 0.066982; visual mesh filename=../../../manipulator/x5/meshes/link1.obj
- added link link2, mass 1.0795; collision box size=0.22 0.06 0.05; collision cylinder length=0.06 radius=0.03
- added link link3, mass 0.54534; collision box size=0.19 0.05 0.04; collision cylinder length=0.05 radius=0.028
- added link link4, mass 0.11714; collision cylinder length=0.04 radius=0.03; visual mesh filename=../../../manipulator/x5/meshes/link4.obj
- added link link5, mass 0.63488; collision cylinder length=0.04 radius=0.03; visual mesh filename=../../../manipulator/x5/meshes/link5.obj
- added link link6, mass 0.44089; collision cylinder length=0.06 radius=0.03; visual mesh filename=../../../manipulator/x5/meshes/link6.obj
- added link link7, mass 0.064798; collision box size=0.03 0.004 0.036; collision box size=0.04 0.004 0.0105
- added link link8, mass 0.064798; collision box size=0.03 0.004 0.036; collision box size=0.04 0.004 0.0105
- link FL_calf: geometry collision cylinder length=0.12 radius=0.012; visual mesh filename=../../../quadruped/go2/meshes/calf_0.obj
- link FL_foot: geometry collision sphere radius=0.022; visual mesh filename=../../../quadruped/go2/meshes/foot.obj
- link FL_hip: geometry collision cylinder length=0.04 radius=0.046; visual mesh filename=../../../quadruped/go2/meshes/hip_0.obj
- link FL_thigh: geometry collision box size=0.11 0.0245 0.034; visual mesh filename=../../../quadruped/go2/meshes/thigh_0.obj
- link FR_calf: geometry collision cylinder length=0.12 radius=0.013; visual mesh filename=../../../quadruped/go2/meshes/calf_mirror_0.obj
- link FR_foot: geometry collision sphere radius=0.022; visual mesh filename=../../../quadruped/go2/meshes/foot.obj
- link FR_hip: geometry collision cylinder length=0.04 radius=0.046; visual mesh filename=../../../quadruped/go2/meshes/hip_0.obj
- link FR_thigh: geometry collision box size=0.11 0.0245 0.034; visual mesh filename=../../../quadruped/go2/meshes/thigh_mirror_0.obj
- link RL_calf: geometry collision cylinder length=0.12 radius=0.013; visual mesh filename=../../../quadruped/go2/meshes/calf_0.obj
- link RL_foot: geometry collision sphere radius=0.022; visual mesh filename=../../../quadruped/go2/meshes/foot.obj
- link RL_hip: geometry collision cylinder length=0.04 radius=0.046; visual mesh filename=../../../quadruped/go2/meshes/hip_0.obj
- link RL_thigh: geometry collision box size=0.11 0.0245 0.034; visual mesh filename=../../../quadruped/go2/meshes/thigh_0.obj
- link RR_calf: geometry collision cylinder length=0.12 radius=0.013; visual mesh filename=../../../quadruped/go2/meshes/calf_mirror_0.obj
- link RR_foot: geometry collision sphere radius=0.022; visual mesh filename=../../../quadruped/go2/meshes/foot.obj
- link RR_hip: geometry collision cylinder length=0.04 radius=0.046; visual mesh filename=../../../quadruped/go2/meshes/hip_0.obj
- link RR_thigh: geometry collision box size=0.11 0.0245 0.034; visual mesh filename=../../../quadruped/go2/meshes/thigh_mirror_0.obj
- link base: geometry collision box size=0.3762 0.0935 0.114; visual mesh filename=../../../quadruped/go2/meshes/base_0.obj
Joints:
- added joint joint1: type revolute, parent link0, child link1, origin xyz=0 0 0.0605 rpy=0 0 0, axis 0 0 1, limit lower=-3.14 upper=2.6 effort=100 velocity=1000
- added joint joint2: type revolute, parent link1, child link2, origin xyz=0.02 0 0.04 rpy=0 0 0, axis 0 1 0, limit lower=-0.1 upper=3.6 effort=100 velocity=1000
- added joint joint3: type revolute, parent link2, child link3, origin xyz=-0.264 0 0 rpy=3.1416 0 0, axis 0 1 0, limit lower=0 upper=3.14 effort=100 velocity=1000
- added joint joint4: type revolute, parent link3, child link4, origin xyz=0.245 0 -0.056 rpy=0 0 0, axis 0 1 0, limit lower=-1.3 upper=1.3 effort=100 velocity=1000
- added joint joint5: type revolute, parent link4, child link5, origin xyz=0.06775 0.0005 -0.0865 rpy=0 0 0, axis 0 0 1, limit lower=-1.57 upper=1.57 effort=100 velocity=1000
- added joint joint6: type revolute, parent link5, child link6, origin xyz=0.02895 0 0.0865 rpy=-3.1416 0 0, axis 1 0 0, limit lower=-2.1 upper=2.1 effort=100 velocity=1000
- added joint joint7: type prismatic, parent link6, child link7, origin xyz=0.08657 0.024896 -0.0002436 rpy=0 0 0, axis 0 1 0, limit lower=0 upper=0.044 effort=100 velocity=1000
- added joint joint8: type prismatic, parent link6, child link8, origin xyz=0.08657 -0.0249 -0.00024366 rpy=0 0 0, axis 0 -1 0, limit lower=0 upper=0.044 effort=100 velocity=1000, mimic joint=joint7 multiplier=1 offset=0
- added joint x5_mount_joint: type revolute, parent base, child link0, origin xyz=0.1 0 0.07 rpy=0 0 0

Commit message: feat: add go2 x5 usd

File: quadruped_manipulator/go2_x5/urdf/go2_x5.urdf (robot description, URDF)
Before this commit: robot go2, 38 links, 37 joints
Links:
- link FL_calf: geometry collision box size=0.024 0.024 0.12; visual mesh filename=../meshes/calf_0.obj
- link FL_calflower: geometry collision box size=0.022 0.022 0.065
- link FL_calflower1: geometry collision box size=0.031 0.031 0.03
- link FR_calf: geometry collision box size=0.026 0.026 0.12; visual mesh filename=../meshes/calf_mirror_0.obj
- link FR_calflower: geometry collision box size=0.022 0.022 0.065
- link FR_calflower1: geometry collision box size=0.031 0.031 0.03
- link RL_calf: geometry collision box size=0.026 0.026 0.12; visual mesh filename=../meshes/calf_0.obj
- link RL_calflower: geometry collision box size=0.022 0.022 0.065
- link RL_calflower1: geometry collision box size=0.031 0.031 0.03
- link RR_calf: geometry collision box size=0.026 0.026 0.12; visual mesh filename=../meshes/calf_mirror_0.obj
- link RR_calflower: geometry collision box size=0.022 0.022 0.065
- link RR_calflower1: geometry collision box size=0.031 0.031 0.03

File: quadruped_manipulator/go2_x5/urdf/go2_x5_fixed_gripper.urdf (robot description, URDF)
Before this commit: robot go2, 39 links, 38 joints
Links:
- link FL_calf: geometry collision box size=0.024 0.024 0.12; visual mesh filename=../meshes/calf_0.obj
- link FL_calflower: geometry collision box size=0.022 0.022 0.065
- link FL_calflower1: geometry collision box size=0.031 0.031 0.03
- link FR_calf: geometry collision box size=0.026 0.026 0.12; visual mesh filename=../meshes/calf_mirror_0.obj
- link FR_calflower: geometry collision box size=0.022 0.022 0.065
- link FR_calflower1: geometry collision box size=0.031 0.031 0.03
- link RL_calf: geometry collision box size=0.026 0.026 0.12; visual mesh filename=../meshes/calf_0.obj
- link RL_calflower: geometry collision box size=0.022 0.022 0.065
- link RL_calflower1: geometry collision box size=0.031 0.031 0.03
- link RR_calf: geometry collision box size=0.026 0.026 0.12; visual mesh filename=../meshes/calf_mirror_0.obj
- link RR_calflower: geometry collision box size=0.022 0.022 0.065
- link RR_calflower1: geometry collision box size=0.031 0.031 0.03
