Commit message: fix: replace cylinder geometries with box geometries in go2.urdf

File: quadruped/go2/urdf/go2.urdf (robot description, URDF)
Before this commit: robot go2, 29 links, 28 joints
Links:
- link FL_calf: geometry collision box size=0.024 0.024 0.12; visual mesh filename=../meshes/calf_0.obj
- link FL_calflower: geometry collision box size=0.022 0.022 0.065
- link FL_calflower1: geometry collision box size=0.031 0.031 0.03
- link FR_calf: geometry collision box size=0.026 0.026 0.12; visual mesh filename=../meshes/calf_mirror_0.obj
- link FR_calflower: geometry collision box size=0.022 0.022 0.065
- link FR_calflower1: geometry collision box size=0.031 0.031 0.03
- link Head_upper: geometry collision box size=0.09 0.09 0.09
- link RL_calf: geometry collision box size=0.026 0.026 0.12; visual mesh filename=../meshes/calf_0.obj
- link RL_calflower: geometry collision box size=0.022 0.022 0.065
- link RL_calflower1: geometry collision box size=0.031 0.031 0.03
- link RR_calf: geometry collision box size=0.026 0.026 0.12; visual mesh filename=../meshes/calf_mirror_0.obj
- link RR_calflower: geometry collision box size=0.022 0.022 0.065
- link RR_calflower1: geometry collision box size=0.031 0.031 0.03
