Commit message: feat: 修改相机连接的URDF结构，更新相机关节的父链接

File: manipulator/piper_l/urdf/piper_l_camera435.urdf (robot description, URDF)
Before this commit: robot piper_l, 15 links, 14 joints
Links:
- removed link camera_bottom_screw_frame
Joints:
- removed joint camera_joint
- joint camera_link_joint: parent camera_bottom_screw_frame -> d435_camera_link
