Commit message: feat: 修改cabinet碰撞体体积

File: object/cabinet/urdf/cabinet.urdf (robot description, URDF)
Before this commit: robot link_robot, 5 links, 4 joints
Links:
- link door_1: geometry collision box size=0.009 0.012 0.110; collision box size=0.014 0.274 0.503
- link drawer_1: geometry collision box size=0.007 0.234 0.110; collision box size=0.008 0.101 0.010
- link drawer_2: geometry collision box size=0.007 0.233 0.112; collision box size=0.008 0.095 0.008
- link drawer_3: geometry collision box size=0.007 0.234 0.140; collision box size=0.008 0.096 0.008
